Commit message: rapp lab vis stuff

File: docker/hw/urdf_override/profiles/bare/tm12s.urdf.xacro (robot description, xacro)
@@ -8,5 +8,5 @@
     <xacro:tm12s_ros2_control name="FakeSystem" initial_positions_file="$(arg initial_positions_file)"/>
     <!-- ==================== PEDESTAL POLE ==================== -->
-    <!-- 580mm tall central pole supporting the robot; 150mm diameter -->
+    <!-- 580mm tall central base supporting the robot; 450mm x 450mm square top -->
     <!-- Extends downward from the robot base (base link is at top of pole) -->
     <joint name="pole_joint" type="fixed">
@@ -18,5 +18,5 @@
         <visual>
             <geometry>
-                <cylinder length="0.58" radius="0.075"/>
+                <box size="0.45 0.45 0.58"/>
             </geometry>
             <material name="pole_gray">
@@ -26,5 +26,5 @@
         <collision>
             <geometry>
-                <cylinder length="0.58" radius="0.075"/>
+                <box size="0.45 0.45 0.58"/>
             </geometry>
         </collision>

File: docker/hw/urdf_override/profiles/team1/tm12s.urdf.xacro (robot description, xacro)
@@ -8,5 +8,5 @@
     <xacro:tm12s_ros2_control name="FakeSystem" initial_positions_file="$(arg initial_positions_file)"/>
     <!-- ==================== PEDESTAL POLE ==================== -->
-    <!-- 580mm tall central pole supporting the robot; 150mm diameter -->
+    <!-- 580mm tall central base supporting the robot; 450mm x 450mm square top -->
     <!-- Extends downward from the robot base (base link is at top of pole) -->
     <joint name="pole_joint" type="fixed">
@@ -18,5 +18,5 @@
         <visual>
             <geometry>
-                <cylinder length="0.58" radius="0.075"/>
+                <box size="0.45 0.45 0.58"/>
             </geometry>
             <material name="pole_gray">
@@ -26,5 +26,5 @@
         <collision>
             <geometry>
-                <cylinder length="0.58" radius="0.075"/>
+                <box size="0.45 0.45 0.58"/>
             </geometry>
         </collision>
